Commit message: Adds inertial parameters to URDF file; fix upper limit at joint 4

File: franka_description/panda_arm_hand.urdf (robot description, URDF)
Before this commit: robot panda, 12 links, 11 joints
Links:
- link panda_hand: mass None -> 0.68
- link panda_leftfinger: mass None -> 0.01
- link panda_link0: mass None -> 3.06
- link panda_link1: mass None -> 2.34
- link panda_link2: mass None -> 2.36
- link panda_link3: mass None -> 2.38
- link panda_link4: mass None -> 2.43
- link panda_link5: mass None -> 3.5
- link panda_link6: mass None -> 1.47
- link panda_link7: mass None -> 0.45
- link panda_rightfinger: mass None -> 0.01
Joints:
- joint panda_joint4: limit lower=-3.0718 upper=0.0873 effort=87 velocity=2.1750 -> lower=-3.0718 upper=-0.0698 effort=87 velocity=2.1750
